Commit message: Rebuild rover URDF-first and generate SDF, calm the drive

File: open_vins/ov_rover_sim/urdf/rover.urdf (robot description, URDF)
Before this commit: robot ov_rover, 9 links, 8 joints
Links:
- link base_link: mass None -> 2.0; geometry collision box size=0.40 0.26 0.15; visual box size=0.40 0.26 0.15
- link cam0_link: geometry visual box size=0.04 0.04 0.04
- link cam1_link: geometry visual box size=0.04 0.04 0.04
- link wheel_front_left_link: mass None -> 0.2; geometry collision cylinder length=0.04 radius=0.08; visual cylinder length=0.04 radius=0.08
- link wheel_front_right_link: mass None -> 0.2; geometry collision cylinder length=0.04 radius=0.08; visual cylinder length=0.04 radius=0.08
- link wheel_rear_left_link: mass None -> 0.2; geometry collision cylinder length=0.04 radius=0.08; visual cylinder length=0.04 radius=0.08
- link wheel_rear_right_link: mass None -> 0.2; geometry collision cylinder length=0.04 radius=0.08; visual cylinder length=0.04 radius=0.08

Commit message: Calm the rover model: torque, mass, contacts

File: open_vins/ov_rover_sim/urdf/rover.urdf (robot description, URDF)
Before this commit: robot ov_rover, 9 links, 8 joints
Links:
- link base_link: mass 2.0 -> 2.5
- link wheel_front_left_link: mass 0.2 -> 0.35
- link wheel_front_right_link: mass 0.2 -> 0.35
- link wheel_rear_left_link: mass 0.2 -> 0.35
- link wheel_rear_right_link: mass 0.2 -> 0.35
